File: pcb/solenoid_driver/solenoid_driver.kicad_sch (KiCad schematic)
At the start: 49 parts, among them J11 OUT1/2, J12 OUT3/4, J13 OUT5/6, J14 OUT7/8, J21 OUT1/2, J22 OUT3/4, J23 OUT5/6, J24 OUT7/8, J31 OUT1/2, J32 OUT3/4, J33 OUT5/6, J34 OUT7/8, J41 OUT1/2, J42 OUT3/4, J43 OUT5/6, J44 OUT7/8, J51 OUT1/2, J52 OUT3/4, J53 OUT5/6, J54 OUT7/8, J61 OUT1/2, J62 OUT3/4, J63 OUT5/6, J64 OUT7/8, J70 12V-IN, J71 CASC-IN, J72 CASC-OUT, U11 74HC595, U12 ULN2803A, U21 74HC595, U22 ULN2803A, U31 74HC595, U32 ULN2803A, U41 74HC595, U42 ULN2803A, U51 74HC595, U52 ULN2803A, U61 74HC595, U62 ULN2803A

Commit message: PCB: trim to 4 cells (3-board plan); place cells + Edge.Cuts (120x66mm); flip top-row terminals mouths-outboard
Parts:
- removed C51, C61: 100nF, Capacitor_THT:C_Disc_D8.0mm_W5.0mm_P5.00mm, symbol Device:C
- removed J51, J61: OUT1/2, TerminalBlock_CUI:TerminalBlock_CUI_TB007-508-02_1x02_P5.08mm_Horizontal, symbol Connector:Screw_Terminal_01x02
- removed J52, J62: OUT3/4, TerminalBlock_CUI:TerminalBlock_CUI_TB007-508-02_1x02_P5.08mm_Horizontal, symbol Connector:Screw_Terminal_01x02
- removed J53, J63: OUT5/6, TerminalBlock_CUI:TerminalBlock_CUI_TB007-508-02_1x02_P5.08mm_Horizontal, symbol Connector:Screw_Terminal_01x02
- removed J54, J64: OUT7/8, TerminalBlock_CUI:TerminalBlock_CUI_TB007-508-02_1x02_P5.08mm_Horizontal, symbol Connector:Screw_Terminal_01x02
- removed U51, U61: 74HC595, Package_DIP:DIP-16_W7.62mm, symbol 74xx:74HC595
- removed U52, U62: ULN2803A, Package_DIP:DIP-18_W7.62mm, symbol Transistor_Array:ULN2803A
Connections:
- net CASC4 is gone; now on net DATA_OUT: U41.9 (QH')
Other:
- moved on the sheet: C41, CB1, CB2, CB3, J41, J42, J43, J44, J70, J71, J72, R1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
